File: level_shifter.kicad_sch (KiCad schematic)
At the start: 13 parts, among them U11 74LVC8T245, U12 74AVC4T245, U13 74LVC8T245

Commit message: fixup some hierarchical buses
Connections:
- net DATAuWire_1: no longer U11.20 (B2)
- net DATAuWire_2: no longer U13.20 (B2)
- net CLKuWire_1 renamed uW1.CLK
- net CLKuWire_2 renamed uW2.CLK
- net LEuWire_1 renamed uW1.LE
- net LEuWire_2 renamed uW2.LE
- new net uW1.DATA: U11.20 (B2)
- new net uW2.DATA: U13.20 (B2)
Changed lines of the file:
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@@
 		(comment 1 "Pedro Rodriguez")
+	)
+	(bus_alias "uW"
+		(members "CLK" "DATA" "LE")
 	)
 	(text "Set as A(fpga)->B(board)"
@@
 		)
 	)
-	(label "LEuWire_2"
+	(label "uW2.LE"
 		(at 58.42 43.18 180)
 		(effects
@@
 		)
 	)
-	(label "DATAuWire_2"
-		(at 166.37 59.69 0)
-		(effects
-			(font
-				(size 1.27 1.27)
-			)
-			(justify left bottom)
-		)
-	)
 	(label "FMC_ADC_DOUT"
 		(at 219.71 157.48 0)
@@
 		)
 	)
+	(label "uW1.CLK"
+		(at 82.55 54.61 180)
+		(effects
+			(font
+				(size 1.27 1.27)
+			)
+			(justify right bottom)
+		)
+	)
 	(label "FMC_ADC_~{CS}"
 		(at 219.71 152.4 0)
@@
 		)
 	)
-	(label "CLKuWire_2"
-		(at 166.37 54.61 0)
-		(effects
-			(font
-				(size 1.27 1.27)
-			)
-			(justify left bottom)
-		)
-	)
 	(label "FMC_CLKuWire_1"
 		(at 219.71 127 0)
@@
 		)
 	)
+	(label "uW2.DATA"
+		(at 175.26 59.69 180)
+		(effects
+			(font
+				(size 1.27 1.27)
+			)
+			(justify right bottom)
+		)
+	)
 	(label "FMC_DATAuWire_1"
 		(at 219.71 129.54 0)
@@
 		)
 	)
-	(label "CLKuWire_2"
+	(label "uW2.CLK"
 		(at 58.42 38.1 180)
 		(effects
@@
 		)
 	)
-	(label "CLKuWire_1"
+	(label "uW1.CLK"
 		(at 58.42 26.67 180)
 		(effects
@@
 		)
 	)
-	(label "DATAuWire_2"
+	(label "uW2.DATA"
 		(at 58.42 40.64 180)
 		(effects
@@
 		)
 	)
-	(label "DATAuWire_1"
-		(at 74.93 59.69 0)
-		(effects
-			(font
-				(size 1.27 1.27)
-			)
-			(justify left bottom)
+	(label "uW2.CLK"
+		(at 175.26 54.61 180)
+		(effects
+			(font
+				(size 1.27 1.27)
+			)
+			(justify right bottom)
 		)
 	)
@@
 		)
 	)
-	(label "LEuWire_1"
-		(at 74.93 64.77 0)
-		(effects
-			(font
-				(size 1.27 1.27)
-			)
-			(justify left bottom)
+	(label "uW1.DATA"
+		(at 82.55 59.69 180)
+		(effects
+			(font
+				(size 1.27 1.27)
+			)
+			(justify right bottom)
 		)
 	)
@@
 		)
 	)
-	(label "CLKuWire_1"
-		(at 74.93 54.61 0)
-		(effects
-			(font
-				(size 1.27 1.27)
-			)
-			(justify left bottom)
-		)
-	)
-	(label "LEuWire_2"
-		(at 166.37 64.77 0)
-		(effects
-			(font
-				(size 1.27 1.27)
-			)
-			(justify left bottom)
-		)
-	)
 	(label "ADC_DIN"
 		(at 58.42 54.61 180)
@@
 		)
 	)
-	(label "DATAuWire_1"
+	(label "uW2.LE"
+		(at 173.99 64.77 180)
+		(effects
+			(font
+				(size 1.27 1.27)
+			)
+			(justify right bottom)
+		)
+	)
+	(label "uW1.DATA"
 		(at 58.42 29.21 180)
 		(effects
@@
 		)
 	)
-	(label "LEuWire_1"
+	(label "uW1.LE"
+		(at 82.55 64.77 180)
+		(effects
+			(font
+				(size 1.27 1.27)
+			)
+			(justify right bottom)
+		)
+	)
+	(label "uW1.LE"
 		(at 58.42 31.75 180)
 		(effects
@@
 		)
 	)
-	(hierarchical_label "{RF_CLK_Control_2}"
+	(hierarchical_label "uW2{uW}"
 		(shape bidirectional)
 		(at 34.29 34.29 180)
@@
 		)
 	)
-	(hierarchical_label "{RF_CLK_Control_1}"
+	(hierarchical_label "uW1{uW}"
 		(shape bidirectional)
 		(at 34.29 22.86 180)
