File: eeprom.kicad_sch (KiCad schematic)
At the start: 9 parts, among them J4 WP Jumper, U9 AT24C64D

Commit message: Draft Schematic Revision
Schematic should be in good shape.
Meta-data and BOM need to be finished.
Very rough layout was started to floorplan out main parts and to see if we have room.
Parts:
- renumbered C36 to C32, J4 to J5, R7 to R10, R8 to R11, R9 to R12, R10 to R13, R5 to R8, R6 to R9, U9 to U12
Changed lines of the file:
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@@
 		(on_board yes)
 		(dnp no)
-		(property "Reference" "R5"
+		(property "Reference" "R8"
 			(at 63.5 55.88 90)
 			(effects
@@
 			(project "rf-input-fmc"
 				(path "/1719e569-47c8-4fa0-8523-9c9686ef0dba/b67143af-be65-48ce-8e48-a6da90939d69"
-					(reference "R5")
+					(reference "R8")
 					(unit 1)
 				)
@@
 		(on_board yes)
 		(dnp no)
-		(property "Reference" "R8"
+		(property "Reference" "R11"
 			(at 114.3 46.99 0)
 			(effects
@@
 			(project "rf-input-fmc"
 				(path "/1719e569-47c8-4fa0-8523-9c9686ef0dba/b67143af-be65-48ce-8e48-a6da90939d69"
-					(reference "R8")
+					(reference "R11")
 					(unit 1)
 				)
@@
 		(on_board yes)
 		(dnp no)
-		(property "Reference" "#PWR029"
+		(property "Reference" "#PWR042"
 			(at 113.03 76.2 0)
 			(effects
@@
 			(project "rf-input-fmc"
 				(path "/1719e569-47c8-4fa0-8523-9c9686ef0dba/b67143af-be65-48ce-8e48-a6da90939d69"
-					(reference "#PWR029")
+					(reference "#PWR042")
 					(unit 1)
 				)
@@
 		(on_board yes)
 		(dnp no)
-		(property "Reference" "U9"
+		(property "Reference" "U12"
 			(at 76.2 50.8 0)
 			(effects
@@
 			(project "rf-input-fmc"
 				(path "/1719e569-47c8-4fa0-8523-9c9686ef0dba/b67143af-be65-48ce-8e48-a6da90939d69"
-					(reference "U9")
+					(reference "U12")
 					(unit 1)
 				)
@@
 		(on_board yes)
 		(dnp no)
-		(property "Reference" "C36"
+		(property "Reference" "C32"
 			(at 87.63 43.18 0)
 			(effects
@@
 			(project "rf-input-fmc"
 				(path "/1719e569-47c8-4fa0-8523-9c9686ef0dba/b67143af-be65-48ce-8e48-a6da90939d69"
-					(reference "C36")
+					(reference "C32")
 					(unit 1)
 				)
@@
 		(on_board yes)
 		(dnp no)
-		(property "Reference" "#PWR027"
+		(property "Reference" "#PWR041"
 			(at 100.33 76.2 0)
 			(effects
@@
 			(project "rf-input-fmc"
 				(path "/1719e569-47c8-4fa0-8523-9c9686ef0dba/b67143af-be65-48ce-8e48-a6da90939d69"
-					(reference "#PWR027")
+					(reference "#PWR041")
 					(unit 1)
 				)
@@
 		(on_board yes)
 		(dnp no)
-		(property "Reference" "R9"
+		(property "Reference" "R12"
 			(at 132.715 52.07 0)
 			(effects
@@
 			(project "rf-input-fmc"
 				(path "/1719e569-47c8-4fa0-8523-9c9686ef0dba/b67143af-be65-48ce-8e48-a6da90939d69"
-					(reference "R9")
+					(reference "R12")
 					(unit 1)
 				)
@@
 		(on_board yes)
 		(dnp no)
-		(property "Reference" "R7"
+		(property "Reference" "R10"
 			(at 80.01 63.5 90)
 			(effects
@@
 			(project "rf-input-fmc"
 				(path "/1719e569-47c8-4fa0-8523-9c9686ef0dba/b67143af-be65-48ce-8e48-a6da90939d69"
-					(reference "R7")
+					(reference "R10")
 					(unit 1)
 				)
@@
 		(on_board yes)
 		(dnp no)
-		(property "Reference" "R6"
+		(property "Reference" "R9"
 			(at 73.66 58.42 90)
 			(effects
@@
 			(project "rf-input-fmc"
 				(path "/1719e569-47c8-4fa0-8523-9c9686ef0dba/b67143af-be65-48ce-8e48-a6da90939d69"
-					(reference "R6")
+					(reference "R9")
 					(unit 1)
 				)
@@
 		(on_board yes)
 		(dnp no)
-		(property "Reference" "J4"
+		(property "Reference" "J5"
 			(at 121.92 63.5 0)
 			(effects
@@
 			(project "rf-input-fmc"
 				(path "/1719e569-47c8-4fa0-8523-9c9686ef0dba/b67143af-be65-48ce-8e48-a6da90939d69"
-					(reference "J4")
+					(reference "J5")
 					(unit 1)
 				)
@@
 		(on_board yes)
 		(dnp no)
-		(property "Reference" "R10"
+		(property "Reference" "R13"
 			(at 140.335 52.07 0)
 			(effects
@@
 			(project "rf-input-fmc"
 				(path "/1719e569-47c8-4fa0-8523-9c9686ef0dba/b67143af-be65-48ce-8e48-a6da90939d69"
-					(reference "R10")
+					(reference "R13")
 					(unit 1)
 				)
@@
 		(on_board yes)
 		(dnp no)
-		(property "Reference" "#PWR026"
+		(property "Reference" "#PWR040"
 			(at 95.25 54.61 0)
 			(effects
@@
 			(project "rf-input-fmc"
 				(path "/1719e569-47c8-4fa0-8523-9c9686ef0dba/b67143af-be65-48ce-8e48-a6da90939d69"
-					(reference "#PWR026")
-					(unit 1)
-				)
+					(reference "#PWR040")
+					(unit 1)
+				)

Commit message: add copyright/license
Other:
- company: Osprey DCS -> SPDX-FileCopyrightText: 2025 Osprey DCS
Changed lines of the file:
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@@
 		(date "2025-10-01")
 		(rev "0.1")
-		(company "Osprey DCS")
-		(comment 1 "Pedro Rodriguez")
+		(company "SPDX-FileCopyrightText: 2025 Osprey DCS")
+		(comment 1 "SPDX-License-Identifier: CERN-OHL-S-2.0+")
 	)
 	(rectangle

Commit message: Changed ADC and removed Level Shifter
- Changed ADC to ADS7253
- Removed Level Shifters
- Change paper size to US standard sizes for printing
- removed 3d models
- Changed SMA clock input to a 2 pin ISORATE connector
- Floor planned out the PCB layout with the new parts
Parts:
- renumbered C32 to C33, J5 to J4, R12 to R10, R13 to R11, R8 to R6, R9 to R7, R10 to R8, R11 to R9, U12 to U10
Other:
- note removed: "EEPROM"
- moved on the sheet: C33, J4, R10, R11, R6, R7, R8, R9, U10

Commit message: Final Schmatic Draft
-Changed ADC
-Changed Digital IO Translator
-Updated all MPNs
- Reannoted Schematic
- Updated Design Document
- Added new Datasheet Document
Parts:
- renumbered R6 to R10, R7 to R11, R8 to R12, R9 to R13, R10 to R14, R11 to R15, U10 to U9
Changed lines of the file:
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@@
 		(on_board yes)
 		(dnp no)
-		(property "Reference" "R6"
+		(property "Reference" "R10"
 			(at 101.6 97.79 90)
 			(effects
@@
 			(project "rf-input-fmc"
 				(path "/1719e569-47c8-4fa0-8523-9c9686ef0dba/b67143af-be65-48ce-8e48-a6da90939d69"
-					(reference "R6")
+					(reference "R10")
 					(unit 1)
 				)
@@
 		(on_board yes)
 		(dnp no)
-		(property "Reference" "R9"
+		(property "Reference" "R13"
 			(at 152.4 88.9 0)
 			(effects
@@
 			(project "rf-input-fmc"
 				(path "/1719e569-47c8-4fa0-8523-9c9686ef0dba/b67143af-be65-48ce-8e48-a6da90939d69"
-					(reference "R9")
+					(reference "R13")
 					(unit 1)
 				)
@@
 		(on_board yes)
 		(dnp no)
-		(property "Reference" "U10"
+		(property "Reference" "U9"
 			(at 114.3 92.71 0)
 			(effects
@@
 			(project "rf-input-fmc"
 				(path "/1719e569-47c8-4fa0-8523-9c9686ef0dba/b67143af-be65-48ce-8e48-a6da90939d69"
-					(reference "U10")
+					(reference "U9")
 					(unit 1)
 				)
@@
 		(on_board yes)
 		(dnp no)
-		(property "Reference" "R10"
+		(property "Reference" "R14"
 			(at 170.815 93.98 0)
 			(effects
@@
 			(project "rf-input-fmc"
 				(path "/1719e569-47c8-4fa0-8523-9c9686ef0dba/b67143af-be65-48ce-8e48-a6da90939d69"
-					(reference "R10")
+					(reference "R14")
 					(unit 1)
 				)
@@
 		(on_board yes)
 		(dnp no)
-		(property "Reference" "R8"
+		(property "Reference" "R12"
 			(at 118.11 105.41 90)
 			(effects
@@
 			(project "rf-input-fmc"
 				(path "/1719e569-47c8-4fa0-8523-9c9686ef0dba/b67143af-be65-48ce-8e48-a6da90939d69"
-					(reference "R8")
+					(reference "R12")
 					(unit 1)
 				)
@@
 		(on_board yes)
 		(dnp no)
-		(property "Reference" "R7"
+		(property "Reference" "R11"
 			(at 111.76 100.33 90)
 			(effects
@@
 			(project "rf-input-fmc"
 				(path "/1719e569-47c8-4fa0-8523-9c9686ef0dba/b67143af-be65-48ce-8e48-a6da90939d69"
-					(reference "R7")
+					(reference "R11")
 					(unit 1)
 				)
@@
 		(on_board yes)
 		(dnp no)
-		(property "Reference" "R11"
+		(property "Reference" "R15"
 			(at 178.435 93.98 0)
 			(effects
@@
 			(project "rf-input-fmc"
 				(path "/1719e569-47c8-4fa0-8523-9c9686ef0dba/b67143af-be65-48ce-8e48-a6da90939d69"
-					(reference "R11")
-					(unit 1)
-				)
+					(reference "R15")
+					(unit 1)
+				)

Commit message: Schematic updates
- Changed Connecters to MMCX
- Added Test points on clocks and data buses
- Added attenuation before the RF input level detection IC to better keep the recommended input within its linear range
- Added a low pass filter at the input of the RF input level detection IC
- grounded the thermal pad of the ADC
- added some additional decoupling caps in for the clock splitter chip (to be in line with what is on Zest)
Parts:
- added TP21, TP22: TestPoint, TestPoint:TestPoint_Pad_D1.0mm, symbol Connector:TestPoint
- renumbered J4 to J19
Connections:
- net SCL: now also TP22.1
- net SDA: now also TP21.1
Changed lines of the file:
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@@
+	)
+	(junction
+		(at 187.96 99.06)
+		(diameter 0)
+		(color 0 0 0 0)
 	)
 	(junction
@@
 	)
 	(junction
+		(at 187.96 101.6)
+		(diameter 0)
+		(color 0 0 0 0)
+	)
+	(junction
 		(at 138.43 81.28)
 		(diameter 0)
@@
 	(wire
 		(pts
-			(xy 175.26 101.6) (xy 181.61 101.6)
+			(xy 175.26 101.6) (xy 187.96 101.6)
+		)
+		(stroke
+			(width 0)
+			(type default)
+		)
+	)
+	(wire
+		(pts
+			(xy 187.96 99.06) (xy 191.77 99.06)
 		)
 		(stroke
@@
 	(wire
 		(pts
-			(xy 167.64 99.06) (xy 181.61 99.06)
+			(xy 167.64 99.06) (xy 187.96 99.06)
+		)
+		(stroke
+			(width 0)
+			(type default)
+		)
+	)
+	(wire
+		(pts
+			(xy 187.96 101.6) (xy 191.77 101.6)
 		)
 		(stroke
@@
 	(hierarchical_label "SDA"
 		(shape bidirectional)
-		(at 181.61 99.06 0)
+		(at 191.77 99.06 0)
 		(effects
 			(font
@@
 	(hierarchical_label "SCL"
 		(shape input)
-		(at 181.61 101.6 0)
+		(at 191.77 101.6 0)
 		(effects
 			(font
@@
 			)
 			(justify right)
+		)
+	)
+	(symbol
+		(lib_id "Connector:TestPoint")
+		(at 187.96 99.06 0)
+		(unit 1)
+		(exclude_from_sim no)
+		(in_bom yes)
+		(on_board yes)
+		(dnp no)
+		(property "Reference" "TP21"
+			(at 185.928 93.726 0)
+			(effects
+				(font
+					(size 1.27 1.27)
+				)
+				(justify left)
+			)
+		)
+		(property "Value" "TestPoint"
+			(at 189.2299 93.98 90)
+			(effects
+				(font
+					(size 1.27 1.27)
+				)
+				(justify left)
+				(hide yes)
+			)
+		)
+		(property "Footprint" "TestPoint:TestPoint_Pad_D1.0mm"
+			(at 193.04 99.06 0)
+			(effects
+				(font
+					(size 1.27 1.27)
+				)
+				(hide yes)
+			)
+		)
+		(property "Datasheet" "~"
+			(at 193.04 99.06 0)
+			(effects
+				(font
+					(size 1.27 1.27)
+				)
+				(hide yes)
+			)
+		)
+		(property "Description" "test point"
+			(at 187.96 99.06 0)
+			(effects
+				(font
+					(size 1.27 1.27)
+				)
+				(hide yes)
+			)
+		)
+		(pin "1"
+		)
+		(instances
+			(project "rf-input-fmc"
+				(path "/1719e569-47c8-4fa0-8523-9c9686ef0dba/b67143af-be65-48ce-8e48-a6da90939d69"
+					(reference "TP21")
+					(unit 1)
+				)
+			)
+		)
+	)
+	(symbol
+		(lib_id "Connector:TestPoint")
+		(at 187.96 101.6 180)
+		(unit 1)
+		(exclude_from_sim no)
+		(in_bom yes)
+		(on_board yes)
+		(dnp no)
+		(property "Reference" "TP22"
+			(at 190.246 107.188 0)
+			(effects
+				(font
+					(size 1.27 1.27)
+				)
+				(justify left)
+			)
+		)
+		(property "Value" "TestPoint"
+			(at 186.6901 106.68 90)
+			(effects
+				(font
+					(size 1.27 1.27)
+				)
+				(justify left)
+				(hide yes)
+			)
+		)
+		(property "Footprint" "TestPoint:TestPoint_Pad_D1.0mm"
+			(at 182.88 101.6 0)
+			(effects
+				(font
+					(size 1.27 1.27)
+				)
+				(hide yes)
+			)
+		)
+		(property "Datasheet" "~"
+			(at 182.88 101.6 0)
+			(effects
+				(font
+					(size 1.27 1.27)
+				)
+				(hide yes)
+			)
+		)
+		(property "Description" "test point"
+			(at 187.96 101.6 0)
+			(effects
+				(font
+					(size 1.27 1.27)
+				)
+				(hide yes)
+			)
+		)
+		(pin "1"
+		)
+		(instances
+			(project "rf-input-fmc"
+				(path "/1719e569-47c8-4fa0-8523-9c9686ef0dba/b67143af-be65-48ce-8e48-a6da90939d69"
+					(reference "TP22")
+					(unit 1)
+				)
+			)
 		)
 	)
@@
 		(on_board yes)
 		(dnp no)
-		(property "Reference" "J4"
+		(property "Reference" "J19"
 			(at 160.02 105.41 0)
 			(effects
@@
 			(project "rf-input-fmc"
 				(path "/1719e569-47c8-4fa0-8523-9c9686ef0dba/b67143af-be65-48ce-8e48-a6da90939d69"
-					(reference "J4")
+					(reference "J19")
 					(unit 1)
 				)

Commit message: Updated BOM of all parts
Updated BOM of all parts
-added supplier & supplier part number to all parts
- fixed many issues with part including:R5-R8,C34,C35,C24, R10-R15

Changed filter C36&C37 to 15nF (keep COG & 0603, but changes filter cutoff to 3.8kHz|was 12kHz)
Changed bulk Caps to 22uF (was 47uF) to get a Cap with enough voltage headroom at 12V while 0805
Changed C31 to be a bulk 10uF cap
Parts:
- C33: MPN CC0603KRX7R7BB105 -> GCM188R71E105KA64D; Manufacturer YAGEO -> Murata Electronics; Supplier (none) -> Digikey; Supplier Part Number (none) -> 490-10673-1-ND
- J19: Supplier (none) -> Digikey; Supplier Part Number (none) -> 952-2261-ND
- R10, R11, R12, R14, R15: MPN RC0603FR-074K42L -> RC0603FR-134K75L; Manufacturer YAGEO -> Yageo; Supplier (none) -> Digikey; Supplier Part Number (none) -> 311-4.42KHRCT-ND
- R13: MPN RC0603FR-0711K5L -> RC0603FR-0711K5L; Manufacturer YAGEO -> Yageo; Supplier (none) -> Digikey; Supplier Part Number (none) -> 311-11.5KHRCT-ND
- TP21, TP22: now left out of the parts list
- U9: Supplier (none) -> Digikey; Supplier Part Number (none) -> AT24C64D-SSHM-TCT-ND

Commit message: Final Draft for prototype run
- Updated CLK mapping to FMC
	 - Now Output 12 goes to M2C CLK instead of a GBT CLK
	 - Outputs 0, 4, 8 have moved
	 - all CLK now have polarity swapped at the FMC pin
		 - CLK signals maintain normal polarity through the CLK distribution chip but are now ALL swapped between the CLK Distribution IC output and the FMC pins
	- Added a monitor output on Output13 (J20)
- Moved decoupling caps to bottom of LCB in many places
- Standardized the area to the right of the FMC to use as a future template
- Moved board specific test points and function to the left
- Added an additional bypass cap on U8
- Tied the front two mounting hole (H3 &H4) to GND
- changed H2 to be a slotted hole
	- This allows for mounting in the FMC slot on Marble where to the mounting hole is shifted by ~4mil
- Add Serial Number area and Board title
- Cleaned up all silkscreen and Fab layers
- Changed J1 & J2 to SMA
	- Added 3d model (from manufacture) to footprint
-  Moved many of the major layout blocks to allow for other changes in this commit
- Added power planes for many major and minor distributed power rails
- pulled back power planes from input connectors
- Fixed all ERC & DRC errors/warnings
Parts:
- removed TP21, TP22: TestPoint, TestPoint:TestPoint_Pad_D1.0mm, symbol Connector:TestPoint
Changed lines of the file:
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@@
-	)
-	(junction
-		(at 187.96 99.06)
-		(diameter 0)
-		(color 0 0 0 0)
 	)
 	(junction
@@
 	)
 	(junction
-		(at 187.96 101.6)
-		(diameter 0)
-		(color 0 0 0 0)
-	)
-	(junction
 		(at 138.43 81.28)
 		(diameter 0)
@@
 	(wire
 		(pts
-			(xy 175.26 101.6) (xy 187.96 101.6)
-		)
-		(stroke
-			(width 0)
-			(type default)
-		)
-	)
-	(wire
-		(pts
-			(xy 187.96 99.06) (xy 191.77 99.06)
+			(xy 175.26 101.6) (xy 191.77 101.6)
 		)
 		(stroke
@@
 	(wire
 		(pts
-			(xy 167.64 99.06) (xy 187.96 99.06)
-		)
-		(stroke
-			(width 0)
-			(type default)
-		)
-	)
-	(wire
-		(pts
-			(xy 187.96 101.6) (xy 191.77 101.6)
+			(xy 167.64 99.06) (xy 191.77 99.06)
 		)
 		(stroke
@@
 		)
 	)
-	(symbol
-		(lib_id "Connector:TestPoint")
-		(at 187.96 99.06 0)
-		(unit 1)
-		(exclude_from_sim no)
-		(in_bom no)
-		(on_board yes)
-		(dnp no)
-		(property "Reference" "TP21"
-			(at 185.928 93.726 0)
-			(effects
-				(font
-					(size 1.27 1.27)
-				)
-				(justify left)
-			)
-		)
-		(property "Value" "TestPoint"
-			(at 189.2299 93.98 90)
-			(effects
-				(font
-					(size 1.27 1.27)
-				)
-				(justify left)
-				(hide yes)
-			)
-		)
-		(property "Footprint" "TestPoint:TestPoint_Pad_D1.0mm"
-			(at 193.04 99.06 0)
-			(effects
-				(font
-					(size 1.27 1.27)
-				)
-				(hide yes)
-			)
-		)
-		(property "Datasheet" "~"
-			(at 193.04 99.06 0)
-			(effects
-				(font
-					(size 1.27 1.27)
-				)
-				(hide yes)
-			)
-		)
-		(property "Description" "test point"
-			(at 187.96 99.06 0)
-			(effects
-				(font
-					(size 1.27 1.27)
-				)
-				(hide yes)
-			)
-		)
-		(property "Supplier" ""
-			(at 187.96 99.06 0)
-			(effects
-				(font
-					(size 1.27 1.27)
-				)
-				(hide yes)
-			)
-		)
-		(property "Supplier Part Number" ""
-			(at 187.96 99.06 0)
-			(effects
-				(font
-					(size 1.27 1.27)
-				)
-				(hide yes)
-			)
-		)
-		(pin "1"
-		)
-		(instances
-			(project "rf-input-fmc"
-				(path "/1719e569-47c8-4fa0-8523-9c9686ef0dba/b67143af-be65-48ce-8e48-a6da90939d69"
-					(reference "TP21")
-					(unit 1)
-				)
-			)
-		)
-	)
-	(symbol
-		(lib_id "Connector:TestPoint")
-		(at 187.96 101.6 180)
-		(unit 1)
-		(exclude_from_sim no)
-		(in_bom no)
-		(on_board yes)
-		(dnp no)
-		(property "Reference" "TP22"
-			(at 190.246 107.188 0)
-			(effects
-				(font
-					(size 1.27 1.27)
-				)
-				(justify left)
-			)
-		)
-		(property "Value" "TestPoint"
-			(at 186.6901 106.68 90)
-			(effects
-				(font
-					(size 1.27 1.27)
-				)
-				(justify left)
-				(hide yes)
-			)
-		)
-		(property "Footprint" "TestPoint:TestPoint_Pad_D1.0mm"
-			(at 182.88 101.6 0)
-			(effects
-				(font
-					(size 1.27 1.27)
-				)
-				(hide yes)
-			)
-		)
-		(property "Datasheet" "~"
-			(at 182.88 101.6 0)
-			(effects
-				(font
-					(size 1.27 1.27)
-				)
-				(hide yes)
-			)
-		)
-		(property "Description" "test point"
-			(at 187.96 101.6 0)
-			(effects
-				(font
-					(size 1.27 1.27)
-				)
-				(hide yes)
-			)
-		)
-		(property "Supplier" ""
-			(at 187.96 101.6 0)
-			(effects
-				(font
-					(size 1.27 1.27)
-				)
-				(hide yes)
-			)
-		)
-		(property "Supplier Part Number" ""
-			(at 187.96 101.6 0)
-			(effects
-				(font
-					(size 1.27 1.27)
-				)
-				(hide yes)
-			)
-		)
-		(pin "1"
-		)
-		(instances
-			(project "rf-input-fmc"
-				(path "/1719e569-47c8-4fa0-8523-9c9686ef0dba/b67143af-be65-48ce-8e48-a6da90939d69"
-					(reference "TP22")
-					(unit 1)
-				)
-			)
-		)
-	)
