File: clk-input-fmc.kicad_sch (KiCad schematic)
At the start: 2 parts

Commit message: Changed Title Blocks to Version 1.0
- changed title blocks
- changed silkscreen to add version number
Other:
- title: RF Input FMC Board -> Clock Input FMC Board
Changed lines of the file:
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@@
 	(paper "USLetter")
 	(title_block
-		(title "RF Input FMC Board")
-		(date "2025-10-16")
-		(rev "0.2")
+		(title "Clock Input FMC Board")
+		(date "2026-05-20")
+		(rev "1.0")
 		(company "SPDX-FileCopyrightText: 2025 Osprey DCS")
 		(comment 1 "SPDX-License-Identifier: CERN-OHL-S-2.0+")
@@
 		)
 		(instances
-			(project "rf-input-fmc"
+			(project "clk-input-fmc"
 				(path "/1719e569-47c8-4fa0-8523-9c9686ef0dba"
 					(page "3")
@@
 		)
 		(instances
-			(project "rf-input-fmc"
+			(project "clk-input-fmc"
 				(path "/1719e569-47c8-4fa0-8523-9c9686ef0dba"
 					(page "6")
@@
 		)
 		(instances
-			(project "rf-input-fmc"
+			(project "clk-input-fmc"
 				(path "/1719e569-47c8-4fa0-8523-9c9686ef0dba"
 					(page "2")
@@
 		)
 		(instances
-			(project "rf-input-fmc"
+			(project "clk-input-fmc"
 				(path "/1719e569-47c8-4fa0-8523-9c9686ef0dba"
 					(page "8")
@@
 		)
 		(instances
-			(project "rf-input-fmc"
+			(project "clk-input-fmc"
 				(path "/1719e569-47c8-4fa0-8523-9c9686ef0dba"
 					(page "7")
@@
 		)
 		(instances
-			(project "rf-input-fmc"
+			(project "clk-input-fmc"
 				(path "/1719e569-47c8-4fa0-8523-9c9686ef0dba"
 					(page "5")
@@
 		)
 		(instances
-			(project "rf-input-fmc"
+			(project "clk-input-fmc"
 				(path "/1719e569-47c8-4fa0-8523-9c9686ef0dba"
 					(page "4")
